Commit message: Sub and Pub matlab scripts

File: urdf/phantom_description_gazebo.xacro (robot description, xacro)
@@ -6,10 +6,8 @@
   <!-- END - Include -->
   <!-- Robot description -->
-  <link name="base_link">
-  </link>
-  <joint name="joint_name" type="fixed">
-    <parent link="base_link"/>
+  <link name="world"/>  <!-- Base link from Gazebo-->
+  <joint name="fixed" type="fixed"> <!-- Joint to fix the base so it does not move-->
+    <parent link="world"/>
     <child link="${link_00_name}"/>
-    <origin xyz="0.0 0.0 0.0" rpy="0.0 0.0 0.0"/>
   </joint>
   <xacro:m_link_mesh name="${link_00_name}"
